Commit message: BREAKING CHANGES: changing repo name

File: celluleflexible/ros_ws/src/Yaskawa_hc10/hc10_ros/urdf/hc10_for_env.urdf (robot description, URDF)
Before this commit: robot motoman_hc10, 8 links, 7 joints
Links:
- removed link base_link
- removed link link_1_s
- removed link link_2_l
- removed link link_3_u
- removed link link_4_r
- removed link link_5_b
- removed link link_6_t
- removed link tool0
Joints:
- removed joint joint_1_s
- removed joint joint_2_l
- removed joint joint_3_u
- removed joint joint_4_r
- removed joint joint_5_b
- removed joint joint_6_t
- removed joint joint_6_t-tool0

File: celluleflexible/ros_ws/src/Yaskawa_hc10/hc10_ros/urdf/hc10_with_env.xacro (robot description, xacro)
@@ -1,18 +1,20 @@
 <?xml version="1.0" ?>
-<robot name="motoman_hc10" xmlns:xacro="http://www.ros.org/wiki/xacro" >
+<robot name="robotic_platform" xmlns:xacro="http://www.ros.org/wiki/xacro" >
+    <!-- loading urdf -->
     <xacro:include filename="$(find hc10_ros)/urdf/materials.xacro" />
-    <link name="world" />
     <xacro:include filename="$(find hc10_ros)/urdf/table.xacro" />
     <xacro:include filename="$(find hc10_ros)/urdf/hc10_for_env.urdf" />
     <xacro:include filename="$(find hc10_ros)/urdf/walls.xacro" />
-    <joint name="walls_joint" type="fixed">
+    <!-- linking every robots to world and workspaces -->
+    <link name="world" />
+    <joint name="world_walls_joint" type="fixed">
         <parent link="world" />
         <child link="walls_link" />
     </joint>
-    <joint name="table_joint" type="fixed">
+    <joint name="wolrd_table_joint" type="fixed">
         <parent link="world" />
         <child link="table_link" />
     </joint>
-    <joint name="link-base" type="fixed">
+    <joint name="table_yaska_base_link" type="fixed">
         <origin rpy="0 0 0" xyz="0 0 0.6376" />
         <parent link="table_link" />
