Commit message: feat: correcting errors

File: celluleflexible/ros_ws/src/Staubli_rx60b/rx60b_support/urdf/rx60.urdf.xacro (robot description, xacro)
@@ -2,5 +2,5 @@
 <robot name="rx60" xmlns:xacro="http://ros.org/wiki/xacro">
   <!-- Import transmission and gazebo elements -->
-  <xacro:include filename="$(find rx60b_description)/urdf/rx60.transmission.xacro"/>
+  <xacro:include filename="$(find rx60b_support)/urdf/rx60.transmission.xacro"/>
   <!-- Links -->
   <xacro:macro name="staubli" params="prefix">
@@ -18,5 +18,5 @@
         <origin xyz="0 0 0" rpy="0 0 0"/>
         <geometry>
-          <mesh filename="package://rx60b_description/meshes/base.dae" scale="1 1 1"/>
+          <mesh filename="package://rx60b_support/meshes/base.dae" scale="1 1 1"/>
         </geometry>
       </visual>
@@ -47,5 +47,5 @@
         <origin xyz="0 0 0" rpy="0 0 0"/>
         <geometry>
-          <mesh filename="package://rx60b_description/meshes/shoulder.dae" scale="1 1 1"/>
+          <mesh filename="package://rx60b_support/meshes/shoulder.dae" scale="1 1 1"/>
         </geometry>
       </visual>
@@ -82,5 +82,5 @@
         <origin xyz="0 0 0" rpy="0 0 1.5707963"/>
         <geometry>
-          <mesh filename="package://rx60b_description/meshes/arm.dae" scale="1 1 1"/>
+          <mesh filename="package://rx60b_support/meshes/arm.dae" scale="1 1 1"/>
         </geometry>
       </visual>
@@ -105,5 +105,5 @@
         <origin xyz="0 0 0" rpy="3.1415926 0 1.5707963"/>
         <geometry>
-          <mesh filename="package://rx60b_description/meshes/elbow.dae" scale="1 1 1"/>
+          <mesh filename="package://rx60b_support/meshes/elbow.dae" scale="1 1 1"/>
         </geometry>
       </visual>
@@ -128,5 +128,5 @@
         <origin xyz="0 0 0" rpy="0 0 0"/>
         <geometry>
-          <mesh filename="package://rx60b_description/meshes/forearm.dae" scale="1 1 1"/>
+          <mesh filename="package://rx60b_support/meshes/forearm.dae" scale="1 1 1"/>
         </geometry>
       </visual>
@@ -163,5 +163,5 @@
         <origin xyz="0 0 0" rpy="3.1415926 0 1.5707963"/>
         <geometry>
-          <mesh filename="package://rx60b_description/meshes/wrist.dae" scale="1 1 1"/>
+          <mesh filename="package://rx60b_support/meshes/wrist.dae" scale="1 1 1"/>
         </geometry>
       </visual>
@@ -186,5 +186,5 @@
         <origin xyz="0 0 0" rpy="0 0 0"/>
         <geometry>
-          <mesh filename="package://rx60b_description/meshes/tool.dae" scale="1 1 1"/>
+          <mesh filename="package://rx60b_support/meshes/tool.dae" scale="1 1 1"/>
         </geometry>
       </visual>

File: celluleflexible/ros_ws/src/robotic_platform_moveit/urdf/robotic_platform_env.xacro (robot description, xacro)
@@ -7,5 +7,5 @@
     <xacro:include filename="$(find hc10_ros)/urdf/walls.xacro" />
     <xacro:include filename="$(find kuka_kr6_support)/urdf/kr6r700sixx.urdf"/>
-    <xacro:include filename="$(find rx60b_description)/urdf/rx60.urdf.xacro"/>
+    <xacro:include filename="$(find rx60b_support)/urdf/rx60.urdf.xacro"/>
     <!-- define prefix to avoid name conflict between joints -->
     <xacro:yaska prefix="yaska4" />
