Commit message: feat: added end effector to yaska4

File: celluleflexible/ros_ws/src/Yaskawa_hc10/yaskawa4/urdf/hc10_with_env.xacro (robot description, xacro)
@@ -6,4 +6,5 @@
     <xacro:include filename="$(find yaskawa4)/urdf/hc10_for_env.urdf" />
     <xacro:include filename="$(find yaskawa4)/urdf/walls.xacro" />
+    <xacro:include filename="$(find yaskawa4)/urdf/pince.xacro"/>
     <xacro:yaska prefix="yaska4" />
     <!-- linking every robots to world and workspaces -->
@@ -13,5 +14,5 @@
         <child link="walls_link" />
     </joint>
-    <joint name="wolrd_table_joint" type="fixed">
+    <joint name="world_table_joint" type="fixed">
         <parent link="world" />
         <child link="table_link" />
@@ -22,3 +23,8 @@
         <child link="yaska4_base_link" />
     </joint>
+    <joint name="end_effector" type="fixed" >
+        <origin rpy="-1.5708 0 0" xyz="0 0 0" />
+        <parent link="yaska4_tool0" />
+        <child link="adaptater_plate_link" />
+    </joint>
 </robot>

File: celluleflexible/ros_ws/src/Yaskawa_hc10/yaskawa4/urdf/materials.xacro (robot description, xacro)
@@ -4,3 +4,6 @@
   <color rgba="0.700 0.700 0.700 1.000"/>
 </material>
+<material name="dark_gray">
+  <color rgba="0.3 0.3 0.3 1.000"/>
+</material>
 </robot>
