Commit message: feat: fix

File: celluleflexible/ros_ws/src/Yaskawa_hc10/yaskawa4/urdf/pince.xacro (robot description, xacro)
@@ -109,5 +109,5 @@
         <parent link="end_effector_link" />
         <child link="adaptater_mors1_link" />
-        <limit effort="1000.0" lower="0" upper="0.037" velocity="0.5"/>
+        <limit effort="1000.0" lower="0" upper="0.035" velocity="0.5"/>
       </joint>
       <!-- ce joint doit être de type prismatique -->
@@ -116,5 +116,5 @@
         <parent link="end_effector_link" />
         <child link="adaptater_mors2_link" />
-        <limit effort="1000.0" lower="0" upper="0.037" velocity="0.5"/>
+        <limit effort="1000.0" lower="0" upper="0.035" velocity="0.5"/>
       </joint>
       <joint name="end_effector_mors1" type="fixed" >
