Commit message: feat: fixing bugs

File: celluleflexible/ros_ws/src/Yaskawa_hc10/yaskawa3/urdf/hc10_with_env.xacro (robot description, xacro)
@@ -1,4 +1,4 @@
 <?xml version="1.0" ?>
-<robot name="motoman_hc10" xmlns:xacro="http://www.ros.org/wiki/xacro" >
+<robot name="yaskawa_3" xmlns:xacro="http://www.ros.org/wiki/xacro" >
     <!-- loading urdf -->
     <xacro:include filename="$(find yaskawa3)/urdf/hc10_for_env.urdf" />

File: celluleflexible/ros_ws/src/Yaskawa_hc10/yaskawa4/urdf/hc10_with_env.xacro (robot description, xacro)
@@ -1,4 +1,4 @@
 <?xml version="1.0" ?>
-<robot name="motoman_hc10" xmlns:xacro="http://www.ros.org/wiki/xacro" >
+<robot name="yaskawa_4" xmlns:xacro="http://www.ros.org/wiki/xacro" >
     <!-- loading urdf -->
     <xacro:include filename="$(find yaskawa4)/urdf/materials.xacro" />
@@ -23,8 +23,8 @@
         <child link="yaska4_base_link" />
     </joint>
-    <joint name="end_effector" type="fixed" >
-        <origin rpy="-1.5708 0 0" xyz="0 0 0" />
+    <joint name="tool_cylinder" type="fixed" >
+        <origin rpy="0 0 0" xyz="0 0 0" />
         <parent link="yaska4_tool0" />
-        <child link="adaptater_plate_link" />
+        <child link="cylinder_link" />
     </joint>
 </robot>

File: celluleflexible/ros_ws/src/Yaskawa_hc10/yaskawa4/urdf/materials.xacro (robot description, xacro)
@@ -7,3 +7,6 @@
   <color rgba="0.3 0.3 0.3 1.000"/>
 </material>
+<material name="white_smoke">
+  <color rgba="0.7607 0.7607 0.7607 1.000"/>
+</material>
 </robot>

File: celluleflexible/ros_ws/src/Yaskawa_hc10/yaskawa4/urdf/pince.xacro (robot description, xacro)
@@ -1,4 +1,18 @@
 <?xml version="1.0" ?>
 <robot name="hand" xmlns:xacro="http://www.ros.org/wiki/xacro">
+    <!-- Ajout des différentes pièces de la pinces / couleurs définies dans le fichier materials.xacro-->
+    <link name="cylinder_link">
+      <visual>
+        <geometry>
+          <mesh filename="package://yaskawa4/meshes/hand/cylinder.stl" scale="1 1 1"/>
+        </geometry>
+        <material name="white_smoke"/>
+      </visual>
+      <collision>
+        <geometry>
+          <mesh filename="package://yaskawa4/meshes/hand/cylinder.stl" scale="1 1 1"/>
+        </geometry>
+      </collision>
+    </link>
     <link name="end_effector_link">
         <visual>
@@ -79,4 +93,10 @@
         </collision>
       </link>
+      <!-- Création des joints  -->
+      <joint name="cylinder_adaptater_plate" type="fixed" >
+        <origin rpy="-1.5708 0 0" xyz="0 0 0.027" />
+        <parent link="cylinder_link" />
+        <child link="adaptater_plate_link" />
+      </joint>
       <joint name="adaptater_plate_end_effector" type="fixed" >
         <origin rpy="0 0 0" xyz="0 -0.012 0" />
@@ -85,14 +105,16 @@
       </joint>
       <!-- ce joint doit être de type prismatique -->
-      <joint name="end_effector_adaptater_mors1" type="fixed" >
+      <joint name="end_effector_adaptater_mors1" type="prismatic" >
         <origin rpy="3.14 0 0" xyz="-0.079 -0.045 0.006" />
         <parent link="end_effector_link" />
         <child link="adaptater_mors1_link" />
+        <limit effort="1000.0" lower="0" upper="0.037" velocity="0.5"/>
       </joint>
       <!-- ce joint doit être de type prismatique -->
-      <joint name="end_effector_adaptater_mors2" type="fixed" >
+      <joint name="end_effector_adaptater_mors2" type="prismatic" >
         <origin rpy="3.14 3.14 0" xyz="0.078 -0.045 -0.023" />
         <parent link="end_effector_link" />
         <child link="adaptater_mors2_link" />
+        <limit effort="1000.0" lower="0" upper="0.037" velocity="0.5"/>
       </joint>
       <joint name="end_effector_mors1" type="fixed" >
