Commit message: feat: updated staubli urdf and execute trajectory script

File: celluleflexible/ros_ws/src/Staubli_tx2_60l/staubli_tx2_60l_moveit/urdf/tx2_60l.xacro (robot description, xacro)
@@ -2,4 +2,10 @@
 <robot name="staubli_tx2_60l" xmlns:xacro="http://wiki.ros.org/xacro">
   <xacro:include filename="$(find staubli_tx2_60l_moveit)/urdf/tx2_60l_macro.xacro"/>
-  <xacro:staubli_tx2_60l prefix=""/>
+  <xacro:include filename="$(find staubli_tx2_60l_moveit)/urdf/pince.xacro" />
+  <xacro:staubli_tx2_60l prefix="staubli_"/>
+  <joint name="tool_end_effector" type="fixed" >
+    <origin rpy="0 0 0" xyz="0 0 0" />
+    <parent link="staubli_tool0" />
+    <child link="end_effector_link" />
+  </joint>
 </robot>
