Commit message: feat: added end effector model for kuka

File: celluleflexible/ros_ws/src/Staubli_tx2_60l/staubli_tx2_60l_moveit/urdf/pince.xacro (robot description, xacro)
@@ -1,22 +1,82 @@
 <?xml version="1.0" ?>
 <robot name="hand" xmlns:xacro="http://www.ros.org/wiki/xacro" >
-  <link name="end_effector_link">
+  <link name="fixation_link">
     <visual>
-      <origin rpy="0 0 0" xyz="0 0 0"/>
       <geometry>
-        <mesh filename="package://staubli_tx2_60l_moveit/meshes/hand/SCHUNK-1372735 EGP 40-N-N-IOL, 00ohne.stl" scale="0.001 0.001 0.001"/>
+        <mesh filename="package://staubli_tx2_60l_moveit/meshes/hand/Outil_Fixation_Bride_Robot_CapteurRef.stl" scale="0.001 0.001 0.001"/>
       </geometry>
-      <!-- <material name="silver"/> -->
+      <material name="silver"/>
     </visual>
     <collision>
-      <origin rpy="0 0 0" xyz="0 0 0"/>
       <geometry>
-        <mesh filename="package://staubli_tx2_60l_moveit/meshes/hand/SCHUNK-1372735 EGP 40-N-N-IOL, 00ohne.stl" scale="0.001 0.001 0.001"/>
+        <mesh filename="package://staubli_tx2_60l_moveit/meshes/hand/Outil_Fixation_Bride_Robot_CapteurRef.stl" scale="0.001 0.001 0.001"/>
       </geometry>
     </collision>
   </link>
-  <!-- <joint name="table_link-base" type="fixed">
-      <parent link="table_link" />
-      <child link="base_table" />
-  </joint> -->
+ <link name="interface_link">
+    <visual>
+      <geometry>
+        <mesh filename="package://staubli_tx2_60l_moveit/meshes/hand/Outil_Pince_Interface_PGNPlus40_EGP40.stl" scale="0.001 0.001 0.001"/>
+      </geometry>
+      <material name="silver"/>
+    </visual>
+    <collision>
+      <geometry>
+        <mesh filename="package://staubli_tx2_60l_moveit/meshes/hand/Outil_Pince_Interface_PGNPlus40_EGP40.stl" scale="0.001 0.001 0.001"/>
+      </geometry>
+    </collision>
+  </link>
+  <link name="end_effector_link">
+    <visual>
+      <geometry>
+        <mesh filename="package://staubli_tx2_60l_moveit/meshes/hand/SCHUNK-0318448 PGN-plus-P 40_ 000.stl" scale="0.001 0.001 0.001"/>
+      </geometry>
+    </visual>
+    <collision>
+      <geometry>
+        <mesh filename="package://staubli_tx2_60l_moveit/meshes/hand/SCHUNK-0318448 PGN-plus-P 40_ 000.stl" scale="0.001 0.001 0.001"/>
+      </geometry>
+    </collision>
+  </link>
+  <link name="mors1_link">
+    <visual>
+      <geometry>
+        <mesh filename="package://staubli_tx2_60l_moveit/meshes/hand/Outil_Pince_Pneumatique_Mors_PGN-Plus-40.stl" scale="0.001 0.001 0.001"/>
+      </geometry>
+    </visual>
+    <collision>
+      <geometry>
+        <mesh filename="package://staubli_tx2_60l_moveit/meshes/hand/Outil_Pince_Pneumatique_Mors_PGN-Plus-40.stl" scale="0.001 0.001 0.001"/>
+      </geometry>
+    </collision>
+  </link>
+  <!--
+  <link name="mors2_link">
+    <visual>
+      <geometry>
+        <mesh filename="package://staubli_tx2_60l_moveit/meshes/hand/Outil_Pince_Pneumatique_Mors_PGN-Plus-40.stl" scale="0.001 0.001 0.001"/>
+      </geometry>
+    </visual>
+    <collision>
+      <geometry>
+        <mesh filename="package://staubli_tx2_60l_moveit/meshes/hand/Outil_Pince_Pneumatique_Mors_PGN-Plus-40.stl" scale="0.001 0.001 0.001"/>
+      </geometry>
+    </collision>
+  </link> -->
+  <!-- Création des joints  -->
+  <joint name="fixation_interface" type="fixed">
+      <origin rpy="3.141592 0 0" xyz="0 0.004 0" />
+      <parent link="fixation_link" />
+      <child link="interface_link" />
+  </joint>
+  <joint name="interface_end_effector" type="fixed">
+      <origin rpy="0 0 0" xyz="0 0.015 0" />
+      <parent link="interface_link" />
+      <child link="end_effector_link" />
+  </joint>
+  <joint name="end_effector_mors1" type="fixed">
+      <origin rpy="0 0 0" xyz="-0.1 0.03 0" />
+      <parent link="end_effector_link" />
+      <child link="mors1_link" />
+  </joint>
 </robot>

File: celluleflexible/ros_ws/src/Staubli_tx2_60l/staubli_tx2_60l_moveit/urdf/tx2_60l.xacro (robot description, xacro)
@@ -1,11 +1,14 @@
 <?xml version="1.0" ?>
 <robot name="staubli_tx2_60l" xmlns:xacro="http://wiki.ros.org/xacro">
+  <!-- loading urdf -->
   <xacro:include filename="$(find staubli_tx2_60l_moveit)/urdf/tx2_60l_macro.xacro"/>
   <xacro:include filename="$(find staubli_tx2_60l_moveit)/urdf/pince.xacro" />
+  <xacro:include filename="$(find staubli_tx2_60l_moveit)/urdf/materials.xacro"/>
   <xacro:staubli_tx2_60l prefix="staubli_"/>
-  <joint name="tool_end_effector" type="fixed" >
-    <origin rpy="0 0 0" xyz="0 0 0" />
+  <!-- linking every robots to world and workspaces -->
+  <joint name="tool_fixation" type="fixed" >
+    <origin rpy="-1.57079 0 0" xyz="0 0 0.00995" />
     <parent link="staubli_tool0" />
-    <child link="end_effector_link" />
+    <child link="fixation_link" />
   </joint>
 </robot>

Commit message: feat: fixed launch files and end effector model of yaskawa3

File: celluleflexible/ros_ws/src/Staubli_tx2_60l/staubli_tx2_60l_moveit/urdf/pince.xacro (robot description, xacro)
@@ -103,21 +103,23 @@
       <child link="end_effector_link" />
   </joint>
-  <joint name="end_effector_adaptater1" type="fixed">
+  <joint name="end_effector_adaptater1" type="prismatic">
       <origin rpy="0 0 0" xyz="0 0 0" />
       <parent link="end_effector_link" />
       <child link="adaptater1_link" />
+      <limit effort="1000.0" lower="0" upper="0.0099" velocity="0.5"/>
   </joint>
-  <joint name="end_effector_adaptater2" type="fixed">
+  <joint name="end_effector_adaptater2" type="prismatic">
       <origin rpy="0 3.1415 0" xyz="0 0 0" />
       <parent link="end_effector_link" />
       <child link="adaptater2_link" />
+      <limit effort="1000.0" lower="0" upper="0.0099" velocity="0.5"/>
   </joint>
   <joint name="adaptater1_mors1" type="fixed">
-      <origin rpy="0 0 0" xyz="-0.0303 0.0247 0.0073" />
+      <origin rpy="0 3.1415 0" xyz="0.0303 0.0247 -0.0073" />
       <parent link="adaptater1_link" />
       <child link="mors1_link" />
   </joint>
   <joint name="adaptater2_mors2" type="fixed">
-      <origin rpy="0 0 0" xyz="-0.0303 0.0247 0.0073" />
+      <origin rpy="0 3.1415 0" xyz="0.0303 0.0247 -0.0073" />
       <parent link="adaptater2_link" />
       <child link="mors2_link" />

File: celluleflexible/ros_ws/src/Yaskawa_hc10/yaskawa3/urdf/hc10_with_env.xacro (robot description, xacro)
@@ -6,4 +6,5 @@
     <xacro:include filename="$(find yaskawa3)/urdf/table.xacro" />
     <xacro:include filename="$(find yaskawa3)/urdf/cell.xacro" />
+    <xacro:include filename="$(find yaskawa3)/urdf/pince.xacro" />
     <xacro:yaska prefix="yaska3" />
     <!-- linking robot to world,workspaces and end-effector -->
@@ -24,3 +25,8 @@
         <child link="yaska3_base_link" />
     </joint>
+    <joint name="tool_adaptater" type="fixed">
+        <origin rpy="-1.57079 0 -1.57079" xyz="0 0 0" />
+        <parent link="yaska3_tool0" />
+        <child link="adaptater_plate_link" />
+    </joint>
 </robot>

File: celluleflexible/ros_ws/src/Yaskawa_hc10/yaskawa4/urdf/hc10_with_env.xacro (robot description, xacro)
@@ -26,5 +26,5 @@
     </joint>
     <joint name="tool_cylinder" type="fixed" >
-        <origin rpy="0 0 0" xyz="0 0 0" />
+        <origin rpy="0 0 -1.57079" xyz="0 0 0" />
         <parent link="yaska4_tool0" />
         <child link="cylinder_link" />
