Commit message: feat: added environment for all robots

File: celluleflexible/ros_ws/src/Kuka_kr6700/kuka_kr6_700sixx_moveit/urdf/cell.xacro (robot description, xacro)
@@ -107,10 +107,10 @@
   </joint>
   <joint name="rail_milieu_rail_tournant1" type="fixed" >
-    <origin rpy="-1.57079 3.14 1.57079" xyz="0.69 0.09 0.003" />
+    <origin rpy="1.57079 0 0" xyz="0.691 -0.09 0.003" />
     <parent link="rail_milieu_link" />
     <child link="rail_tournant1_link" />
   </joint>
   <joint name="rail_milieu_rail_tournant2" type="fixed" >
-    <origin rpy="-1.57079 3.14 0" xyz="-0.651 0.09 0.003" />
+    <origin rpy="1.57079 0 1.57079" xyz="-0.65 -0.09 0.003" />
     <parent link="rail_milieu_link" />
     <child link="rail_tournant2_link" />

File: celluleflexible/ros_ws/src/Kuka_kr6700/kuka_kr6_700sixx_moveit/urdf/kr6r700sixx.xacro (robot description, xacro)
@@ -10,15 +10,15 @@
   <link name="world" />
   <joint name="world_cell" type="fixed">
-      <origin rpy="0 0 0" xyz="0 0.5 0.698"/>
+      <origin rpy="0 0 3.14" xyz="0 0.5 0.698"/>
       <parent link="world" />
       <child link="pieds_cellule_link" />
   </joint>
   <joint name="world_table" type="fixed">
-      <origin rpy="0 0 0" xyz="0.03 0 0.645" />
+      <origin rpy="0 0 0" xyz="-0.03 0 0.645" />
       <parent link="world" />
       <child link="pieds_table_link" />
   </joint>
   <joint name="table_kuka" type="fixed">
-      <origin rpy="0 0 1.57079" xyz="0.25 0 0" />
+      <origin rpy="0 1.57079 1.57079" xyz="0 0 0" />
       <parent link="plateau_table_link" />
       <child link="kuka_base_link" />

File: celluleflexible/ros_ws/src/Kuka_kr6700/kuka_kr6_700sixx_moveit/urdf/table.xacro (robot description, xacro)
@@ -20,5 +20,5 @@
       <origin rpy="0 0 0" xyz="0 0 0"/>
       <geometry>
-        <mesh filename="package://kuka_kr6_700sixx_moveit/meshes/env/plateau_table.stl" scale="0.01 0.01 0.01"/>
+        <mesh filename="package://kuka_kr6_700sixx_moveit/meshes/env/plateau_table_kuka.stl" scale="1 1 1"/>
       </geometry>
       <material name="dark_gray"/>
@@ -27,10 +27,10 @@
       <origin rpy="0 0 0" xyz="0 0 0"/>
       <geometry>
-        <mesh filename="package://kuka_kr6_700sixx_moveit/meshes/env/plateau_table.stl" scale="0.01 0.01 0.01"/>
+        <mesh filename="package://kuka_kr6_700sixx_moveit/meshes/env/plateau_table_kuka.stl" scale="1 1 1"/>
       </geometry>
     </collision>
   </link>
   <joint name="pieds_plateau_table" type="fixed">
-    <origin rpy="0 0 0" xyz="0 0 0.343" />
+    <origin rpy="1.57079 0 0" xyz="0 0 0.343" />
     <parent link="pieds_table_link" />
     <child link="plateau_table_link" />

File: celluleflexible/ros_ws/src/Staubli_tx2_60l/staubli_tx2_60l_moveit/urdf/tx2_60l.xacro (robot description, xacro)
@@ -10,4 +10,19 @@
   <!-- linking robot to world,workspaces and end-effector -->
   <link name="world" />
+  <joint name="world_cell" type="fixed">
+      <origin rpy="0 0 0" xyz="-0.2 0.48 0.698"/>
+      <parent link="world" />
+      <child link="pieds_cellule_link" />
+  </joint>
+  <joint name="world_table" type="fixed">
+      <origin rpy="0 0 0" xyz="0 0 0.645" />
+      <parent link="world" />
+      <child link="pieds_table_link" />
+  </joint>
+  <joint name="table_staubli" type="fixed">
+      <origin rpy="-1.57079 3.14 0" xyz="0.201 0.0075 0.008" />
+      <parent link="plateau_table_staubli_link" />
+      <child link="staubli_base_link" />
+  </joint>
   <joint name="tool_fixation" type="fixed" >
     <origin rpy="-1.57079 0 0" xyz="0 0 0.00995" />

File: celluleflexible/ros_ws/src/Yaskawa_hc10/yaskawa3/urdf/cell.xacro (robot description, xacro)
@@ -1,9 +1,9 @@
 <?xml version="1.0" ?>
 <robot name="env" xmlns:xacro="http://www.ros.org/wiki/xacro" >
-  <link name="cellule_link">
+  <link name="pieds_cellule_link">
     <visual>
       <origin rpy="0 0 0" xyz="0 0 0"/>
       <geometry>
-        <mesh filename="package://yaskawa3/meshes/env/cellule.stl" scale="0.01 0.01 0.01"/>
+        <mesh filename="package://yaskawa3/meshes/env/pieds_cellule.stl" scale="1 1 1"/>
       </geometry>
       <material name="silver"/>
@@ -12,7 +12,107 @@
       <origin rpy="0 0 0" xyz="0 0 0"/>
       <geometry>
-        <mesh filename="package://yaskawa3/meshes/env/cellule.stl" scale="0.01 0.01 0.01"/>
+        <mesh filename="package://yaskawa3/meshes/env/pieds_cellule.stl" scale="1 1 1"/>
       </geometry>
     </collision>
   </link>
+  <link name="ergots1_link">
+    <visual>
+      <origin rpy="0 0 0" xyz="0 0 0"/>
+      <geometry>
+        <mesh filename="package://yaskawa3/meshes/env/ergots.stl" scale="0.001 0.001 0.001"/>
+      </geometry>
+      <material name="dark_gray"/>
+    </visual>
+    <collision>
+      <origin rpy="0 0 0" xyz="0 0 0"/>
+      <geometry>
+        <mesh filename="package://yaskawa3/meshes/env/ergots.stl" scale="0.001 0.001 0.001"/>
+      </geometry>
+    </collision>
+  </link>
+  <link name="ergots2_link">
+    <visual>
+      <origin rpy="0 0 0" xyz="0 0 0"/>
+      <geometry>
+        <mesh filename="package://yaskawa3/meshes/env/ergots.stl" scale="0.001 0.001 0.001"/>
+      </geometry>
+      <material name="dark_gray"/>
+    </visual>
+    <collision>
+      <origin rpy="0 0 0" xyz="0 0 0"/>
+      <geometry>
+        <mesh filename="package://yaskawa3/meshes/env/ergots.stl" scale="0.001 0.001 0.001"/>
+      </geometry>
+    </collision>
+  </link>
+  <link name="rail_milieu_link">
+    <visual>
+      <origin rpy="0 0 0" xyz="0 0 0"/>
+      <geometry>
+        <mesh filename="package://yaskawa3/meshes/env/rail_milieu.stl" scale="0.001 0.001 0.001"/>
+      </geometry>
+      <material name="silver"/>
+    </visual>
+    <collision>
+      <origin rpy="0 0 0" xyz="0 0 0"/>
+      <geometry>
+        <mesh filename="package://yaskawa3/meshes/env/rail_milieu.stl" scale="0.001 0.001 0.001"/>
+      </geometry>
+    </collision>
+  </link>
+  <link name="rail_tournant1_link">
+    <visual>
+      <origin rpy="0 0 0" xyz="0 0 0"/>
+      <geometry>
+        <mesh filename="package://yaskawa3/meshes/env/rail_tournant.stl" scale="0.001 0.001 0.001"/>
+      </geometry>
+      <material name="silver"/>
+    </visual>
+    <collision>
+      <origin rpy="0 0 0" xyz="0 0 0"/>
+      <geometry>
+        <mesh filename="package://yaskawa3/meshes/env/rail_tournant.stl" scale="0.001 0.001 0.001"/>
+      </geometry>
+    </collision>
+  </link>
+  <link name="rail_tournant2_link">
+    <visual>
+      <origin rpy="0 0 0" xyz="0 0 0"/>
+      <geometry>
+        <mesh filename="package://yaskawa3/meshes/env/rail_tournant.stl" scale="0.001 0.001 0.001"/>
+      </geometry>
+      <material name="silver"/>
+    </visual>
+    <collision>
+      <origin rpy="0 0 0" xyz="0 0 0"/>
+      <geometry>
+        <mesh filename="package://yaskawa3/meshes/env/rail_tournant.stl" scale="0.001 0.001 0.001"/>
+      </geometry>
+    </collision>
+  </link>
+  <joint name="pieds_cellule_ergots1" type="fixed" >
+    <origin rpy="0 0 0" xyz="0.111 0.025 0.485" />
+    <parent link="pieds_cellule_link" />
+    <child link="ergots1_link" />
+  </joint>
+  <joint name="pieds_cellule_ergots2" type="fixed" >
+    <origin rpy="0 0 0" xyz="-0.29 0.025 0.485" />
+    <parent link="pieds_cellule_link" />
+    <child link="ergots2_link" />
+  </joint>
+  <joint name="pieds_cellule_rail_milieu" type="fixed" >
+    <origin rpy="0 0 0" xyz="-0.02 0 0.403" />
+    <parent link="pieds_cellule_link" />
+    <child link="rail_milieu_link" />
+  </joint>
+  <joint name="rail_milieu_rail_tournant1" type="fixed" >
+    <origin rpy="-1.57079 3.14 1.57079" xyz="0.69 0.09 0.003" />
+    <parent link="rail_milieu_link" />
+    <child link="rail_tournant1_link" />
+  </joint>
+  <joint name="rail_milieu_rail_tournant2" type="fixed" >
+    <origin rpy="-1.57079 3.14 0" xyz="-0.651 0.09 0.003" />
+    <parent link="rail_milieu_link" />
+    <child link="rail_tournant2_link" />
+  </joint>
 </robot>

File: celluleflexible/ros_ws/src/Yaskawa_hc10/yaskawa3/urdf/hc10_with_env.xacro (robot description, xacro)
@@ -10,15 +10,15 @@
     <link name="world" />
     <joint name="world_cell" type="fixed">
-        <origin rpy="1.5708 0 0" xyz="-0.8 0.15 0.44"/>
+        <origin rpy="0 0 -1.57079" xyz="0.72 0.27 0.698"/>
         <parent link="world" />
-        <child link="cellule_link" />
+        <child link="pieds_cellule_link" />
     </joint>
     <joint name="world_table" type="fixed">
-        <origin rpy="0 0 0" xyz="0 0 0" />
+        <origin rpy="1.57079 0 0" xyz="0 0 0.432"/>
         <parent link="world" />
         <child link="table_link" />
     </joint>
     <joint name="table_yaska3" type="fixed">
-        <origin rpy="0 0 0" xyz="0 0 0.6376" />
+        <origin rpy="-1.57079 0 0" xyz="0.171 0.203 0.181" />
         <parent link="table_link" />
         <child link="yaska3_base_link" />

File: celluleflexible/ros_ws/src/Yaskawa_hc10/yaskawa3/urdf/table.xacro (robot description, xacro)
@@ -5,5 +5,5 @@
       <origin rpy="0 0 0" xyz="0 0 0"/>
       <geometry>
-        <mesh filename="package://yaskawa3/meshes/env/table.stl" scale="0.01 0.01 0.01"/>
+        <mesh filename="package://yaskawa3/meshes/env/table_yaskawa.stl" scale="1 1 1"/>
       </geometry>
       <material name="silver"/>
@@ -12,5 +12,5 @@
       <origin rpy="0 0 0" xyz="0 0 0"/>
       <geometry>
-        <mesh filename="package://yaskawa3/meshes/env/table.stl" scale="0.01 0.01 0.01"/>
+        <mesh filename="package://yaskawa3/meshes/env/table_yaskawa.stl" scale="1 1 1"/>
       </geometry>
     </collision>

File: celluleflexible/ros_ws/src/Yaskawa_hc10/yaskawa4/urdf/hc10_with_env.xacro (robot description, xacro)
@@ -5,19 +5,21 @@
     <xacro:include filename="$(find yaskawa4)/urdf/table.xacro" />
     <xacro:include filename="$(find yaskawa4)/urdf/hc10_for_env.urdf" />
-    <xacro:include filename="$(find yaskawa4)/urdf/walls.xacro" />
+    <xacro:include filename="$(find yaskawa4)/urdf/cell.xacro" />
     <xacro:include filename="$(find yaskawa4)/urdf/pince.xacro"/>
     <xacro:yaska prefix="yaska4" />
    <!-- linking robot to world,workspaces and end-effector -->
     <link name="world" />
-    <joint name="world_walls_joint" type="fixed">
+    <joint name="world_cell" type="fixed">
+        <origin rpy="0 0 0" xyz="-0.29 -0.73 0.698"/>
         <parent link="world" />
-        <child link="walls_link" />
+        <child link="pieds_cellule_link" />
     </joint>
     <joint name="world_table_joint" type="fixed">
+        <origin rpy="1.57079 0 0" xyz="0 0 0.432"/>
         <parent link="world" />
         <child link="table_link" />
     </joint>
     <joint name="link_base" type="fixed">
-        <origin rpy="0 0 0" xyz="0 0 0.6376" />
+        <origin rpy="-1.57079 1.57079 0" xyz="0.171 0.2 0.181" />
         <parent link="table_link" />
         <child link="yaska4_base_link" />

File: celluleflexible/ros_ws/src/Yaskawa_hc10/yaskawa4/urdf/table.xacro (robot description, xacro)
@@ -5,5 +5,5 @@
       <origin rpy="0 0 0" xyz="0 0 0"/>
       <geometry>
-        <mesh filename="package://yaskawa4/meshes/env/table.stl" scale="0.01 0.01 0.01"/>
+        <mesh filename="package://yaskawa4/meshes/env/table_yaskawa.stl" scale="1 1 1"/>
       </geometry>
       <material name="silver"/>
@@ -12,5 +12,5 @@
       <origin rpy="0 0 0" xyz="0 0 0"/>
       <geometry>
-        <mesh filename="package://yaskawa4/meshes/env/table.stl" scale="0.01 0.01 0.01"/>
+        <mesh filename="package://yaskawa4/meshes/env/table_yaskawa.stl" scale="1 1 1"/>
       </geometry>
     </collision>
