Commit message: feat: added environnement for kuka in the urdf

File: celluleflexible/ros_ws/src/Kuka_kr6700/kuka_kr6_700sixx_moveit/urdf/kr6r700sixx.xacro (robot description, xacro)
@@ -4,6 +4,24 @@
   <xacro:include filename="$(find kuka_kr6_700sixx_moveit)/urdf/pince.xacro" />
   <xacro:include filename="$(find kuka_kr6_700sixx_moveit)/urdf/materials.xacro"/>
+  <xacro:include filename="$(find kuka_kr6_700sixx_moveit)/urdf/table.xacro" />
+  <xacro:include filename="$(find kuka_kr6_700sixx_moveit)/urdf/cell.xacro" />
   <xacro:kuka_kr6r700sixx prefix="kuka_"/>
-  <!-- linking every robots to world and workspaces -->
+  <!-- linking robot to world,workspaces and end-effector -->
+  <link name="world" />
+  <joint name="world_cell" type="fixed">
+      <origin rpy="0 0 0" xyz="0 0.5 0.698"/>
+      <parent link="world" />
+      <child link="pieds_cellule_link" />
+  </joint>
+  <joint name="world_table" type="fixed">
+      <origin rpy="0 0 0" xyz="0.03 0 0.645" />
+      <parent link="world" />
+      <child link="pieds_table_link" />
+  </joint>
+  <joint name="table_kuka" type="fixed">
+      <origin rpy="0 0 1.57079" xyz="0.25 0 0" />
+      <parent link="plateau_table_link" />
+      <child link="kuka_base_link" />
+  </joint>
   <joint name="tool_adapater_plate" type="fixed" >
     <origin rpy="0 0 1.57079" xyz="0 0 0.0045" />

File: celluleflexible/ros_ws/src/Staubli_tx2_60l/staubli_tx2_60l_moveit/urdf/tx2_60l.xacro (robot description, xacro)
@@ -5,6 +5,9 @@
   <xacro:include filename="$(find staubli_tx2_60l_moveit)/urdf/pince.xacro" />
   <xacro:include filename="$(find staubli_tx2_60l_moveit)/urdf/materials.xacro"/>
+  <xacro:include filename="$(find staubli_tx2_60l_moveit)/urdf/table.xacro" />
+  <xacro:include filename="$(find staubli_tx2_60l_moveit)/urdf/cell.xacro" />
   <xacro:staubli_tx2_60l prefix="staubli_"/>
-  <!-- linking every robots to world and workspaces -->
+  <!-- linking robot to world,workspaces and end-effector -->
+  <link name="world" />
   <joint name="tool_fixation" type="fixed" >
     <origin rpy="-1.57079 0 0" xyz="0 0 0.00995" />

File: celluleflexible/ros_ws/src/Yaskawa_hc10/yaskawa3/urdf/cell.xacro (robot description, xacro)
@@ -1,9 +1,9 @@
 <?xml version="1.0" ?>
 <robot name="env" xmlns:xacro="http://www.ros.org/wiki/xacro" >
-  <link name="table_link">
+  <link name="cellule_link">
     <visual>
       <origin rpy="0 0 0" xyz="0 0 0"/>
       <geometry>
-        <mesh filename="package://yaskawa4/meshes/env/table.stl" scale="0.01 0.01 0.01"/>
+        <mesh filename="package://yaskawa3/meshes/env/cellule.stl" scale="0.01 0.01 0.01"/>
       </geometry>
       <material name="silver"/>
@@ -12,5 +12,5 @@
       <origin rpy="0 0 0" xyz="0 0 0"/>
       <geometry>
-        <mesh filename="package://yaskawa4/meshes/env/table.stl" scale="0.01 0.01 0.01"/>
+        <mesh filename="package://yaskawa3/meshes/env/cellule.stl" scale="0.01 0.01 0.01"/>
       </geometry>
     </collision>

File: celluleflexible/ros_ws/src/Yaskawa_hc10/yaskawa3/urdf/hc10_with_env.xacro (robot description, xacro)
@@ -2,11 +2,24 @@
 <robot name="yaskawa_3" xmlns:xacro="http://www.ros.org/wiki/xacro" >
     <!-- loading urdf -->
+    <xacro:include filename="$(find yaskawa3)/urdf/materials.xacro" />
     <xacro:include filename="$(find yaskawa3)/urdf/hc10_for_env.urdf" />
+    <xacro:include filename="$(find yaskawa3)/urdf/table.xacro" />
+    <xacro:include filename="$(find yaskawa3)/urdf/cell.xacro" />
     <xacro:yaska prefix="yaska3" />
-    <!-- linking every robots to world and workspaces -->
+    <!-- linking robot to world,workspaces and end-effector -->
     <link name="world" />
-    <joint name="link_base" type="fixed">
+    <joint name="world_cell" type="fixed">
+        <origin rpy="1.5708 0 0" xyz="-0.8 0.15 0.44"/>
+        <parent link="world" />
+        <child link="cellule_link" />
+    </joint>
+    <joint name="world_table" type="fixed">
         <origin rpy="0 0 0" xyz="0 0 0" />
         <parent link="world" />
+        <child link="table_link" />
+    </joint>
+    <joint name="table_yaska3" type="fixed">
+        <origin rpy="0 0 0" xyz="0 0 0.6376" />
+        <parent link="table_link" />
         <child link="yaska3_base_link" />
     </joint>

File: celluleflexible/ros_ws/src/Yaskawa_hc10/yaskawa3/urdf/table.xacro (robot description, xacro)
@@ -5,5 +5,5 @@
       <origin rpy="0 0 0" xyz="0 0 0"/>
       <geometry>
-        <mesh filename="package://yaskawa4/meshes/env/table.stl" scale="0.01 0.01 0.01"/>
+        <mesh filename="package://yaskawa3/meshes/env/table.stl" scale="0.01 0.01 0.01"/>
       </geometry>
       <material name="silver"/>
@@ -12,5 +12,5 @@
       <origin rpy="0 0 0" xyz="0 0 0"/>
       <geometry>
-        <mesh filename="package://yaskawa4/meshes/env/table.stl" scale="0.01 0.01 0.01"/>
+        <mesh filename="package://yaskawa3/meshes/env/table.stl" scale="0.01 0.01 0.01"/>
       </geometry>
     </collision>

File: celluleflexible/ros_ws/src/Yaskawa_hc10/yaskawa4/urdf/hc10_with_env.xacro (robot description, xacro)
@@ -8,5 +8,5 @@
     <xacro:include filename="$(find yaskawa4)/urdf/pince.xacro"/>
     <xacro:yaska prefix="yaska4" />
-    <!-- linking every robots to world and workspaces -->
+   <!-- linking robot to world,workspaces and end-effector -->
     <link name="world" />
     <joint name="world_walls_joint" type="fixed">

Commit message: feat: added trajectory for kuka

File: celluleflexible/ros_ws/src/Kuka_kr6700/kuka_kr6_700sixx_moveit/urdf/kr6r700sixx.xacro (robot description, xacro)
@@ -20,5 +20,5 @@
   </joint>
   <joint name="table_kuka" type="fixed">
-      <origin rpy="0 1.57079 1.57079" xyz="0 0 0" />
+      <origin rpy="1.57079 0 3.1415" xyz="0 0 0" />
       <parent link="plateau_table_link" />
       <child link="kuka_base_link" />

File: celluleflexible/ros_ws/src/Kuka_kr6700/kuka_kr6_700sixx_moveit/urdf/pince.xacro (robot description, xacro)
@@ -89,5 +89,5 @@
     <parent link="KGG_link" />
     <child link="liaison1_link" />
-    <limit effort="1000.0" lower="0" upper="0.03" velocity="0.5"/>
+    <limit effort="1000.0" lower="-0.5" upper="0.031" velocity="0.5"/>
   </joint>
   <joint name="KGG_laison2" type="prismatic" >
@@ -95,5 +95,5 @@
     <parent link="KGG_link" />
     <child link="liaison2_link" />
-    <limit effort="1000.0" lower="0" upper="0.03" velocity="0.5"/>
+    <limit effort="1000.0" lower="-0.5" upper="0.031" velocity="0.5"/>
   </joint>
   <joint name="liason1_mors1" type="fixed" >

File: celluleflexible/ros_ws/src/Kuka_kr6700/kuka_kr6_700sixx_moveit/urdf/table.xacro (robot description, xacro)
@@ -32,5 +32,5 @@
   </link>
   <joint name="pieds_plateau_table" type="fixed">
-    <origin rpy="1.57079 0 0" xyz="0 0 0.343" />
+    <origin rpy="1.57079 0 0" xyz="0.21 0 0.343" />
     <parent link="pieds_table_link" />
     <child link="plateau_table_link" />
