Commit message: feat: position home changed to fit real config

File: celluleflexible/ros_ws/src/Yaskawa_hc10/yaskawa1/urdf/hc10_with_env.xacro (robot description, xacro)
@@ -20,5 +20,5 @@
     </joint>
     <joint name="table_yaska1" type="fixed">
-        <origin rpy="-1.57079 0 0" xyz="0.171 0.203 0.181" />
+        <origin rpy="-1.57079 1.57079 0" xyz="0.171 0.203 0.181" />
         <parent link="table_link" />
         <child link="yaska1_base_link" />

File: celluleflexible/ros_ws/src/Yaskawa_hc10/yaskawa4/urdf/hc10_with_env.xacro (robot description, xacro)
@@ -21,5 +21,5 @@
     </joint>
     <joint name="link_base" type="fixed">
-        <origin rpy="-1.57079 1.57079 0" xyz="0.171 0.2 0.181" />
+        <origin rpy="-1.57079 3.1415 0" xyz="0.171 0.2 0.181" />
         <parent link="table_link" />
         <child link="yaska4_base_link" />
